Commit message: cleans up finger mesh files, fixes bug with finger distance in model

File: svenzva_description/robots/svenzva_arm.xacro (robot description, xacro)
@@ -421,11 +421,11 @@
       velocity="1" />
   </joint>
-  <xacro:revel_finger parent="link_6" finger_number="1" mesh_path="package://svenzva_description/meshes/finger_link_1.STL">
-      <origin xyz="-0.00483282204262809 -0.00411403012500923 0.0206210772714723" rpy="0 0 -3.14159" />
+  <xacro:revel_finger parent="link_6" finger_number="1" mesh_path="package://svenzva_description/meshes/finger_standard.STL">
+      <origin xyz="0 0 -0.00196" rpy="0 0 -3.14159" />
       <axis xyz="0 -1 0" />
   </xacro:revel_finger>
-  <xacro:revel_finger parent="link_6" finger_number="2" mesh_path="package://svenzva_description/meshes/finger_joint_2.STL">
-    <origin xyz="0.00483282233149502 0.00411402197005728 0.020621076918268"    rpy="0 0 -3.14159" />
-    <axis xyz="0 1 0" />
+  <xacro:revel_finger parent="link_6" finger_number="2" mesh_path="package://svenzva_description/meshes/finger_standard.STL">
+      <origin xyz="0 0 -0.00196" rpy="0 0 0" />
+      <axis xyz="0 1 0" />
   </xacro:revel_finger>
   <link name="${end_effector_link_name}"> </link>
