Commit message: many changes in package structure and general driver abilities

File: svenzva_description/robots/svenzva_arm.urdf (robot description, URDF)
Before this commit: robot svenzva_description, 8 links, 7 joints
Joints:
- joint ee_joint: origin xyz=0.015 0 0.15 -> xyz=0 0 0.0
- joint joint_1: limit lower=0.0 upper=6.0 effort=30 velocity=1.0 -> lower=0 upper=6.0 effort=30 velocity=1.0
- joint joint_6: limit lower=-6.0 upper=0.0 effort=30 velocity=1.0 -> lower=0.0 upper=6.0 effort=30 velocity=1.0

Commit message: updated model

File: svenzva_description/robots/svenzva_arm.urdf (robot description, URDF)
Before this commit: robot svenzva_description, 8 links, 7 joints
Links:
- removed link ee_link
- added link link_7, mass 0.0354585256038568; collision mesh filename=package://svenzva_description/meshes/link_7.STL; visual mesh filename=package://svenzva_description/meshes/link_7.STL
- link base_link: mass 0.072364 -> 0.506214468139727
- link link_1: mass 0.176002844262561 -> 0.153541664031025
- link link_2: mass 0.375844350417551 -> 0.281175487770198
- link link_3: mass 0.31163055657781 -> 0.246165133529195
- link link_4: mass 0.227468523944588 -> 0.211922628762084
- link link_5: mass 0.151584942075443 -> 0.164460903684414
- link link_6: mass 0.322937867529949 -> 0.195112141464075
Joints:
- removed joint ee_joint
- added joint joint_7: type prismatic, parent link_6, child link_7, origin xyz=0 0 -0.0573569998840002 rpy=-3.14159265358979 0 -3.14159265358979, axis -1 0 0, limit lower=-0.05 upper=0.05 effort=5 velocity=1.0
- joint joint_1: axis 0 1 0 -> 0 0 1; origin xyz=0.013 0 0.040487 rpy=1.5708 -1.1432E-16 -0.01434 -> xyz=0 0 0.07119999984 rpy=-1.93033535706571E-16 -1.54074395550979E-32 0
- joint joint_2: axis 0 0 -1 -> 0 0 1; origin xyz=0 0.0964625315349195 -0.0233499999819998 rpy=4.09187004857075E-18 -1.3761561334924E-14 1.60002689098321E-18 -> xyz=0.00891249579997938 0 0.09644999999 rpy=1.5707963267949 -1.93033535706571E-16 1.5707963267949
- joint joint_3: axis 0 0 1 -> 0 0 -1; origin xyz=0 0.22669999999 0.0158749999819999 rpy=6.69447407664753E-16 1.6306400674182E-16 -0.00242557244235328 -> xyz=0 0.22770179999 0.00317500840002059 rpy=-3.14159265358979 -2.14461300673676E-15 3.14159265358979
- joint joint_4: axis 0 0 -1.0 -> 0 0 1; origin xyz=0.00912959083561864 0.137721791833396 0.0137499861543416 rpy=-2.36709870890947 1.57079630572147 -2.36079769092609 -> xyz=-0.00165000009395299 0.13769999999 0.00581250408200003 rpy=0 1.5707963267949 0
- joint joint_5: origin xyz=0.00645000003795365 0.1377 -0.00249999436214027 rpy=0 1.5707963267949 0 -> xyz=0.00165000009004705 0.15039999999 -0.00158749994695297 rpy=0 1.5707963267949 0
- joint joint_6: axis 0 0 1 -> 0 0 -1; origin xyz=0.0153032852422354 0.0855005794492288 -0.0126999817460203 rpy=-1.5707963267949 -1.55645636523858 -1.09070333872558E-05 -> xyz=-0.0147500000020004 0.0754999999999999 0.00142499999999982 rpy=1.5707963267949 1.5707963267949 0

Commit message: added colors, ee_link added

File: svenzva_description/robots/svenzva_arm.urdf (robot description, URDF)
Before this commit: robot svenzva_description, 9 links, 8 joints
Joints:
- joint joint_1: axis 0 0 1 -> 0 0 -1
- joint joint_2: axis 0 0 1 -> 0 0 -1
- joint joint_5: axis 0 0 1 -> 0 0 -1
- joint joint_7: type prismatic -> fixed

Commit message: model updated to 4_24 version

File: svenzva_description/robots/svenzva_arm.urdf (robot description, URDF)
Before this commit: robot svenzva_description, 9 links, 8 joints
Links:
- removed link ee_link
- link base_link: mass 0.506214468139727 -> 0.438546009395726; geometry collision mesh filename=package://4_25_urdf6/meshes/base_link.STL; visual mesh filename=package://4_25_urdf6/meshes/base_link.STL
- link link_1: mass 0.153541664031025 -> 0.21227632351697; geometry collision mesh filename=package://4_25_urdf6/meshes/link_1.STL; visual mesh filename=package://4_25_urdf6/meshes/link_1.STL
- link link_2: mass 0.281175487770198 -> 0.293474008383791; geometry collision mesh filename=package://4_25_urdf6/meshes/link_2.STL; visual mesh filename=package://4_25_urdf6/meshes/link_2.STL
- link link_3: mass 0.246165133529195 -> 0.254948895895984; geometry collision mesh filename=package://4_25_urdf6/meshes/link_3.STL; visual mesh filename=package://4_25_urdf6/meshes/link_3.STL
- link link_4: mass 0.211922628762084 -> 0.220706391128874; geometry collision mesh filename=package://4_25_urdf6/meshes/link_4.STL; visual mesh filename=package://4_25_urdf6/meshes/link_4.STL
- link link_5: mass 0.164460903684414 -> 0.163854288137822; geometry collision mesh filename=package://4_25_urdf6/meshes/link_5.STL; visual mesh filename=package://4_25_urdf6/meshes/link_5.STL
- link link_6: mass 0.195112141464075 -> 0.210564848441307; geometry collision mesh filename=package://4_25_urdf6/meshes/link_6.STL; visual mesh filename=package://4_25_urdf6/meshes/link_6.STL
- link link_7: mass 0.0354585256038568 -> 0.0177292628019284; geometry collision mesh filename=package://4_25_urdf6/meshes/link_finger_1.STL; visual mesh filename=package://4_25_urdf6/meshes/link_finger_1.STL
Joints:
- removed joint ee_joint
- joint joint_1: axis 0 0 -1 -> 0 0 1; origin xyz=0 0 0.07119999984 rpy=-1.93033535706571E-16 -1.54074395550979E-32 0 -> xyz=0 0 0.06485 rpy=0 0 -4.404E-17
- joint joint_2: axis 0 0 -1 -> 0 0 1; limit lower=-2.0 upper=2.0 effort=30 velocity=1.0 -> lower=-2 upper=2 effort=30 velocity=1.0; origin xyz=0.00891249579997938 0 0.09644999999 rpy=1.5707963267949 -1.93033535706571E-16 1.5707963267949 -> xyz=0 -0.015113 0.1155 rpy=1.5708 0 4.3282E-16
- joint joint_3: limit lower=-2.0 upper=2.0 effort=30 velocity=1.0 -> lower=-2 upper=2 effort=30 velocity=1.0; origin xyz=0 0.22770179999 0.00317500840002059 rpy=-3.14159265358979 -2.14461300673676E-15 3.14159265358979 -> xyz=0 0.2277 -0.009226 rpy=3.1416 -1.5345E-16 3.1416
- joint joint_4: limit lower=-2.4 upper=2.4 effort=30 velocity=1.0 -> lower=-1.7 upper=1.7 effort=30 velocity=1.0; origin xyz=-0.00165000009395299 0.13769999999 0.00581250408200003 rpy=0 1.5707963267949 0 -> xyz=-0.00165 0.1377 -0.000388 rpy=0 1.5708 0
- joint joint_5: axis 0 0 -1 -> 0 0 1; limit lower=-1.9 upper=1.9 effort=30 velocity=1.0 -> lower=-1.7 upper=1.7 effort=30 velocity=1.0; origin xyz=0.00165000009004705 0.15039999999 -0.00158749994695297 rpy=0 1.5707963267949 0 -> xyz=0.00165 0.1504 -0.0015875 rpy=0 1.5708 0
- joint joint_6: limit lower=0.0 upper=6.0 effort=30 velocity=1.0 -> lower=0 upper=6.0 effort=30 velocity=1.0; origin xyz=-0.0147500000020004 0.0754999999999999 0.00142499999999982 rpy=1.5707963267949 1.5707963267949 0 -> xyz=-0.01475 0.08 0.001425 rpy=1.5708 1.5708 0
- joint joint_7: limit lower=-0.05 upper=0.05 effort=5 velocity=1.0 -> lower=-0.05 upper=0.05 effort=30 velocity=1.0; origin xyz=0 0 -0.0573569998840002 rpy=-3.14159265358979 0 -3.14159265358979 -> xyz=0 0 -0.052509 rpy=3.1416 3.0358E-17 3.1416; type fixed -> prismatic

Commit message: manual modifications in model to match motor zero position

File: svenzva_description/robots/svenzva_arm.urdf (robot description, URDF)
Before this commit: robot revel, 8 links, 7 joints
Joints:
- joint joint_1: axis 0 0 1 -> 0 0 -1; origin xyz=0 0 0.06485 rpy=0 0 -4.404E-17 -> xyz=0 0 0.06485 rpy=0 0 -1.5708
- joint joint_2: axis 0 0 1 -> 0 0 -1
- joint joint_5: axis 0 0 1 -> 0 0 -1
- joint joint_6: origin xyz=-0.01475 0.08 0.001425 rpy=1.5708 1.5708 0 -> xyz=-0.01475 0.08 0.001425 rpy=1.5708 3.14159 0

Commit message: many changes getting compliance smooth, general driver organization and threading, and improvements.

File: svenzva_description/robots/svenzva_arm.urdf (robot description, URDF)
Before this commit: robot revel, 8 links, 7 joints
Links:
- added link ee_link
- link base_link: mass 0.438546009395726 -> 0.774961748747901
- link link_1: mass 0.21227632351697 -> 0.29849024
- link link_2: mass 0.293474008383791 -> 0.327742070931929
- link link_3: mass 0.254948895895984 -> 0.280463750144268
- link link_4: mass 0.220706391128874 -> 0.246221245377158
- link link_6: mass 0.210564848441307 -> 0.251621037329208
- link link_7: mass 0.0177292628019284 -> 0.0478690095652066
Joints:
- added joint ee_joint: type fixed, parent link_6, child ee_link, origin xyz=0 0 0.0

Commit message: general changes. added joint limits to cartesian controller. modified urdf to allow turns in either direction

File: svenzva_description/robots/svenzva_arm.urdf (robot description, URDF)
Before this commit: robot revel, 9 links, 8 joints
Joints:
- joint joint_1: limit lower=0 upper=6.0 effort=30 velocity=1.0 -> lower=-3.14 upper=3.14 effort=30 velocity=1.0

Commit message: modified joint limit for cable mgmt

File: svenzva_description/robots/svenzva_arm.urdf (robot description, URDF)
Before this commit: robot revel, 9 links, 8 joints
Joints:
- joint joint_6: limit lower=0 upper=6.0 effort=30 velocity=1.0 -> lower=1.2 upper=7.8 effort=30 velocity=1.0

Commit message: modified urdf and improved cartesian controller somewhat. orientation z motion is closer to expected behavior

File: svenzva_description/robots/svenzva_arm.urdf (robot description, URDF)
Before this commit: robot revel, 9 links, 8 joints
Links:
- removed link link_7
Joints:
- removed joint joint_7
- joint ee_joint: origin xyz=0 0 -0.1 rpy=3.14159 0 0 -> xyz=0.0 0.08 0 rpy=-1.5708 0 0
- joint joint_2: origin xyz=0 -0.015113 0.1155 rpy=1.5708 0 4.3282E-16 -> xyz=0 -0.015113 0.1155 rpy=1.5708 0 0
- joint joint_3: origin xyz=0 0.2277 -0.009226 rpy=3.1416 -1.5345E-16 3.1416 -> xyz=0 0.2277 -0.009226 rpy=3.1416 0.0 3.1416
- joint joint_5: origin xyz=0.00165 0.1504 -0.0015875 rpy=0 1.5708 0 -> xyz=0.0 0.1504 0.0 rpy=0 1.5708 0
- joint joint_6: axis 0 0 -1 -> 0 1 0; limit lower=0 upper=8.0 effort=30 velocity=1.0 -> effort=100 velocity=100.0; origin xyz=-0.01475 0.08 0.001425 rpy=1.5708 3.14159 0 -> xyz=-0.01877 0.08 0 rpy=0 3.14159 0; type revolute -> continuous

Commit message: changes???

File: svenzva_description/robots/svenzva_arm.urdf (robot description, URDF)
Before this commit: robot revel, 8 links, 7 joints
Joints:
- joint ee_joint: origin xyz=0.0 0.08 0 rpy=-1.5708 0 0 -> xyz=0.0 0 0.08 rpy=0 0 0
- joint joint_2: origin xyz=0 -0.015113 0.1155 rpy=1.5708 0 0 -> xyz=0 0 0.1155 rpy=1.5708 0 0
- joint joint_3: origin xyz=0 0.2277 -0.009226 rpy=3.1416 0.0 3.1416 -> xyz=0 0.2277 0 rpy=3.1416 0.0 3.1416
- joint joint_4: origin xyz=-0.00165 0.1377 -0.000388 rpy=0 1.5708 0 -> xyz=0 0.1377 0 rpy=0 1.5708 0
- joint joint_6: axis 0 1 0 -> 0 0 1; origin xyz=-0.01877 0.08 0 rpy=0 3.14159 0 -> xyz=0 0.08 0 rpy=-1.5807 0 0

Commit message: updated inertial values

File: svenzva_description/robots/svenzva_arm.urdf (robot description, URDF)
Before this commit: robot revel, 8 links, 7 joints
Links:
- link base_link: mass 0.774961748747901 -> 0.6323
- link link_1: mass 0.29849024 -> 0.300074
- link link_2: mass 0.327742070931929 -> 0.38526
- link link_3: mass 0.280463750144268 -> 0.312507
- link link_4: mass 0.246221245377158 -> 0.295819
- link link_5: mass 0.163854288137822 -> 0.1901733
- link link_6: mass 0.251621037329208 -> 0.3029304

Commit message: added separate prismatic fingers

File: svenzva_description/robots/svenzva_arm.urdf (robot description, URDF)
Before this commit: robot revel, 8 links, 7 joints
Links:
- removed link ee_link
- added link link_finger1, mass 0.0478690095652066; collision mesh filename=package://svenzva_description/meshes/finger.STL; visual mesh filename=package://svenzva_description/meshes/finger.STL
- added link link_finger2, mass 0.0478690095652066; collision mesh filename=package://svenzva_description/meshes/finger.STL; visual mesh filename=package://svenzva_description/meshes/finger.STL
Joints:
- removed joint ee_joint
- added joint joint_7: type prismatic, parent link_6, child link_finger1, origin xyz=0 0 -0.052509 rpy=3.1416 3.0358E-17 3.1416, axis -1 0 0, limit lower=0 upper=0.05 effort=30 velocity=1.0
- added joint joint_8: type prismatic, parent link_6, child link_finger2, origin xyz=0 0 -0.052509 rpy=3.1416 3.0358E-17 3.1416, axis -1 0 0, limit lower=-0.05 upper=0.0 effort=30 velocity=1.0

Commit message: new urdf

File: svenzva_description/robots/svenzva_arm.urdf (robot description, URDF)
Before this commit: robot revel, 9 links, 8 joints
Links:
- removed link link_finger1
- removed link link_finger2
- link base_link: mass 0.6323 -> 0.72202
- link link_1: mass 0.300074 -> 0.29504
- link link_2: mass 0.38526 -> 0.33821
- link link_3: mass 0.312507 -> 0.25639
- link link_4: mass 0.295819 -> 0.18149
- link link_5: mass 0.1901733 -> 0.17619
- link link_6: mass 0.3029304 -> 0.23371
Joints:
- removed joint joint_7
- removed joint joint_8
- joint joint_1: limit lower=-3.14 upper=3.14 effort=30 velocity=1.0 -> lower=-3.14 upper=3.14 effort=30 velocity=1; origin xyz=0 0 0.06485 rpy=0 0 -1.5708 -> xyz=0 0 0.0762 rpy=0 0 0
- joint joint_2: limit lower=-2 upper=2 effort=30 velocity=1.0 -> lower=-2 upper=2 effort=30 velocity=1; origin xyz=0 0 0.1155 rpy=1.5708 0 0 -> xyz=-0.007325 0 0.10542 rpy=1.5708 0 -1.5708
- joint joint_3: limit lower=-2.2 upper=2.2 effort=30 velocity=1.0 -> lower=-2.2 upper=2.2 effort=30 velocity=1; origin xyz=0 0.2277 0 rpy=3.1416 0.0 3.1416 -> xyz=0 0.2277 0.00635 rpy=3.1416 -2.0986E-16 3.1416
- joint joint_4: limit lower=-2.0 upper=2.0 effort=30 velocity=1.0 -> lower=-2 upper=2 effort=30 velocity=1; origin xyz=0 0.1377 0 rpy=0 1.5708 0 -> xyz=-0.022225 0.15508 0.0074 rpy=1.5708 2.0986E-16 3.1416
- joint joint_5: axis 0 0 -1 -> 0 0 1; limit lower=-1.7 upper=1.7 effort=30 velocity=1.0 -> lower=-1.7 upper=1.7 effort=30 velocity=1; origin xyz=0.0 0.1504 0.0 rpy=0 1.5708 0 -> xyz=0 0.00165 0.095204 rpy=1.5708 0 3.1416
- joint joint_6: axis 0 0 1 -> 0 0 -1; limit effort=100 velocity=100.0 -> (none); origin xyz=0 0.08 0 rpy=-1.5807 0 0 -> xyz=-0.01475 0.08 0.001425 rpy=1.5708 1.6799E-15 2.9288E-15

Commit message: changed urdf and moveit config

File: svenzva_description/robots/svenzva_arm.urdf (robot description, URDF)
Before this commit: robot svenzva_description, 7 links, 6 joints
Links:
- added link finger_joint_2, mass 0.0220307791071739; collision mesh filename=package://svenzva_description/meshes/finger_joint_2.STL; visual mesh filename=package://svenzva_description/meshes/finger_joint_2.STL
- added link finger_link_1, mass 0.0220307791071739; collision mesh filename=package://svenzva_description/meshes/finger_link_1.STL; visual mesh filename=package://svenzva_description/meshes/finger_link_1.STL
- link base_link: mass 0.72202 -> 0.761337238502044
- link link_1: mass 0.29504 -> 0.295038974095265
- link link_2: mass 0.33821 -> 0.344381379534998
- link link_3: mass 0.25639 -> 0.196650631153951
- link link_4: mass 0.18149 -> 0.171727164051589
- link link_5: mass 0.17619 -> 0.13919813472784
- link link_6: mass 0.23371 -> 0.243320868687054
Joints:
- added joint finger_joint_1: type prismatic, parent link_6, child finger_link_1, origin xyz=0 0 -0.052509 rpy=-3.1416 -1.8964E-18 3.1416, axis 0 1 0, limit lower=0 upper=0.05 effort=0 velocity=0
- added joint finger_joint_2: type prismatic, parent link_6, child finger_joint_2, origin xyz=0 0 -0.052509 rpy=-3.1416 -1.8964E-18 3.1416, axis 0 1 0, limit lower=-0.05 upper=0 effort=0 velocity=0
- joint joint_1: limit lower=-3.14 upper=3.14 effort=30 velocity=1 -> lower=-3.14 upper=3.14 effort=0 velocity=0; origin xyz=0 0 0.0762 rpy=0 0 0 -> xyz=0 0 0.0762 rpy=0 0 -4.404E-17
- joint joint_2: limit lower=-2 upper=2 effort=30 velocity=1 -> lower=-2 upper=2 effort=0 velocity=0
- joint joint_3: limit lower=-2.2 upper=2.2 effort=30 velocity=1 -> lower=-2 upper=2 effort=0 velocity=0
- joint joint_4: limit lower=-2 upper=2 effort=30 velocity=1 -> lower=-5.0 upper=3.867165 effort=0 velocity=0; origin xyz=-0.022225 0.15508 0.0074 rpy=1.5708 2.0986E-16 3.1416 -> xyz=-0.020448 0.11835 0.0083512 rpy=-1.5672 1.5708 0
- joint joint_5: axis 0 0 1 -> 0 0 -1; limit lower=-1.7 upper=1.7 effort=30 velocity=1 -> lower=-1.7 upper=1.7 effort=0 velocity=0; origin xyz=0 0.00165 0.095204 rpy=1.5708 0 3.1416 -> xyz=-0.0010724 -2.0879E-05 0.08245 rpy=1.5708 -0.0035837 -1.5708
- joint joint_6: limit (none) -> lower=-1.565 upper=1.565 effort=0 velocity=0; origin xyz=-0.01475 0.08 0.001425 rpy=1.5708 1.6799E-15 2.9288E-15 -> xyz=-0.014463 0.080052 0.001425 rpy=1.5744 -1.5708 0; type continuous -> revolute

Commit message: fixes merged issues with new urdf. updates moveit.

File: svenzva_description/robots/svenzva_arm.urdf (robot description, URDF)
Before this commit: robot revel, 10 links, 9 joints
Joints:
- joint joint_6: limit lower=3.2 upper=8.8 effort=0 velocity=0 -> lower=-1.6 upper=1.6 effort=0 velocity=0

Commit message: filled in erroneous effort and velocity limits in urdf

File: svenzva_description/robots/svenzva_arm.urdf (robot description, URDF)
Before this commit: robot revel, 10 links, 9 joints
Joints:
- joint finger_joint_1: limit lower=0 upper=0.05 effort=0 velocity=0 -> lower=0 upper=0.05 effort=100 velocity=10
- joint finger_joint_2: limit lower=-0.05 upper=0 effort=0 velocity=0 -> lower=-0.05 upper=0 effort=100 velocity=10
- joint joint_1: limit lower=-3.14 upper=3.14 effort=0 velocity=0 -> lower=-3.14 upper=3.14 effort=100 velocity=10
- joint joint_2: limit lower=-2 upper=2 effort=0 velocity=0 -> lower=-2 upper=2 effort=100 velocity=10
- joint joint_3: limit lower=-2 upper=2 effort=0 velocity=0 -> lower=-2 upper=2 effort=100 velocity=10
- joint joint_4: limit lower=-5 upper=3.867 effort=0 velocity=0 -> lower=-5 upper=3.867 effort=100 velocity=10
- joint joint_5: limit lower=-1.7 upper=1.7 effort=0 velocity=0 -> lower=-1.7 upper=1.7 effort=100 velocity=10
- joint joint_6: limit lower=-1.6 upper=1.6 effort=0 velocity=0 -> lower=-1.6 upper=1.6 effort=100 velocity=10

Commit message: fixes namespace incompatibility between gazebo and moveits expected controller space. incorrect inertial and mass values corrected for link_4 and link_3

File: svenzva_description/robots/svenzva_arm.urdf (robot description, URDF)
Before this commit: robot revel, 10 links, 9 joints
Links:
- link link_3: mass 0.227860881806706 -> 0.285860881806706
- link link_4: mass 0.174540765744632 -> 0.236769
Joints:
- joint joint_4: limit lower=-5 upper=3.867 effort=100 velocity=10 -> lower=-3 upper=3 effort=10 velocity=1

Commit message: added new urdf

File: svenzva_description/robots/svenzva_arm.urdf (robot description, URDF)
Before this commit: robot revel, 10 links, 9 joints
Links:
- link link_4: mass 0.236769 -> 0.197871876004791
- link link_5: mass 0.133021865517638 -> 0.16384; geometry collision mesh filename=package://3_9_18_revel/meshes/link_5.STL; visual mesh filename=package://3_9_18_revel/meshes/link_5.STL
Joints:
- joint joint_4: limit lower=-3 upper=3 effort=10 velocity=1 -> lower=-3.0 upper=3.0 effort=10 velocity=2; origin xyz=-0.022225 0.17977 0.0074 rpy=1.5708 0 -3.1416 -> xyz=0.00317500540000185 0.2037305 0.00740000000000075 rpy=1.5707963267949 1.14512197671461E-15 -3.14159265358979
- joint joint_5: limit lower=-1.7 upper=1.7 effort=100 velocity=10 -> lower=-1.7 upper=1.7 effort=10 velocity=2; origin xyz=0 0.00165 0.07925 rpy=1.5708 0 -3.1416 -> xyz=0.0039474 -0.0021486 0.075895 rpy=1.5708 -1.1102E-16 9.4421E-32

Commit message: changed gripper limits in accordance with offset change

File: svenzva_description/robots/svenzva_arm.urdf (robot description, URDF)
Before this commit: robot revel, 10 links, 9 joints
Joints:
- joint joint_4: axis 0 0 1 -> 0 0 -1
- joint joint_6: limit lower=-1.6 upper=1.6 effort=100 velocity=10 -> lower=0.5 upper=5.5 effort=10 velocity=2; origin xyz=-0.01475 0.08 0.001425 rpy=1.5708 0 0 -> xyz=-0.01475 0.08 0.001425 rpy=1.5708 1.5708 0

Commit message: limit changes

File: svenzva_description/robots/svenzva_arm.urdf (robot description, URDF)
Before this commit: robot revel, 10 links, 9 joints
Joints:
- joint joint_2: limit lower=-2 upper=2 effort=100 velocity=10 -> lower=-2.2 upper=2.2 effort=100 velocity=10
- joint joint_3: limit lower=-2 upper=2 effort=100 velocity=10 -> lower=-2.2 upper=2.2 effort=100 velocity=10
- joint joint_4: limit lower=-3.0 upper=3.0 effort=10 velocity=2 -> lower=-2.5 upper=4.0 effort=10 velocity=2

Commit message: added parameter for enabling velocity checking, added end effector link, tested new ways to find singularities

File: svenzva_description/robots/svenzva_arm.urdf (robot description, URDF)
Before this commit: robot revel, 10 links, 9 joints
Links:
- added link ee_link
Joints:
- added joint ee_joint: type fixed, parent link_6, child ee_link, origin xyz=0 0 -0.05 rpy=3.14159 0 0

Commit message: adds updated urdf.

File: svenzva_description/robots/svenzva_arm.urdf (robot description, URDF)
Before this commit: robot revel, 11 links, 10 joints
Links:
- link base_link: mass 0.722020764728074 -> 0.789077111415677
- link link_1: mass 0.095038974095265 -> 0.285081724446302
- link link_2: mass 0.350557648873674 -> 0.500798339631218
- link link_3: mass 0.285860881806706 -> 0.371611749675941
- link link_4: mass 0.197871876004791 -> 0.186398780121232
- link link_5: mass 0.16384 -> 0.141592490303688; geometry collision mesh filename=package://svenzva_description/meshes/link_5.STL; visual mesh filename=package://svenzva_description/meshes/link_5.STL
- link link_6: mass 0.243320868551208 -> 0.222489248107418
Joints:
- joint joint_1: limit lower=-3.14 upper=3.14 effort=100 velocity=10 -> lower=-3.14 upper=3.14 effort=10 velocity=1; origin xyz=0 0 0.0762 rpy=0 0 0 -> xyz=0 0 0.064752 rpy=0 0 0
- joint joint_2: limit lower=-2.2 upper=2.2 effort=100 velocity=10 -> lower=-2.2 upper=2.2 effort=10 velocity=1; origin xyz=-0.007325 0 0.10542 rpy=1.5708 0 -1.5708 -> xyz=0.00038333 -0.0069353 0.10441 rpy=1.5708 0 0
- joint joint_3: axis 0 0 -1 -> 0 0 1; limit lower=-2.2 upper=2.2 effort=100 velocity=10 -> lower=-2.2 upper=2.2 effort=10 velocity=1; origin xyz=0 0.2277 0.00635 rpy=3.1416 0 3.1416 -> xyz=0 0.2224 0.014294 rpy=0 0 0
- joint joint_4: axis 0 0 -1 -> 0 -1 0; limit lower=-2.5 upper=4.0 effort=10 velocity=2 -> lower=-2.5 upper=4.0 effort=10 velocity=1; origin xyz=0.00317500540000185 0.2037305 0.00740000000000075 rpy=1.5707963267949 1.14512197671461E-15 -3.14159265358979 -> xyz=0 0.19605 -0.015019 rpy=0 0 0
- joint joint_5: axis 0 0 -1 -> 0 1 0; limit lower=-1.7 upper=1.7 effort=10 velocity=2 -> lower=-1.7 upper=1.7 effort=10 velocity=1; origin xyz=0.0039474 -0.0021486 0.075895 rpy=1.5708 -1.1102E-16 9.4421E-32 -> xyz=0 0.08375 0.0040438 rpy=-1.5708 0 0
- joint joint_6: limit lower=0.5 upper=5.5 effort=10 velocity=2 -> lower=0.5 upper=5.5 effort=10 velocity=1; origin xyz=-0.01475 0.08 0.001425 rpy=1.5708 1.5708 0 -> xyz=0 -0.019119 0.082 rpy=3.1416 0 1.5708
