Commit message: urdf update

File: svenzva_description/robots/svenzva_arm.urdf (robot description, URDF)
Before this commit: robot revel, 11 links, 10 joints
Links:
- link base_link: mass 0.789077111415677 -> 0.673945611735726; geometry collision mesh filename=package://4_24_18_revel/meshes/base_link.STL; visual mesh filename=package://4_24_18_revel/meshes/base_link.STL
- link link_1: mass 0.285081724446302 -> 0.386092665970672; geometry collision mesh filename=package://4_24_18_revel/meshes/link_1.STL; visual mesh filename=package://4_24_18_revel/meshes/link_1.STL
- link link_2: mass 0.500798339631218 -> 0.63194; geometry collision mesh filename=package://4_24_18_revel/meshes/link_2.STL; visual mesh filename=package://4_24_18_revel/meshes/link_2.STL
- link link_3: mass 0.371611749675941 -> 0.37014; geometry collision mesh filename=package://4_24_18_revel/meshes/link_3.STL; visual mesh filename=package://4_24_18_revel/meshes/link_3.STL
- link link_4: mass 0.186398780121232 -> 0.208577727676899; geometry collision mesh filename=package://4_24_18_revel/meshes/link_4.STL; visual mesh filename=package://4_24_18_revel/meshes/link_4.STL
- link link_5: mass 0.141592490303688 -> 0.198143515414093; geometry collision mesh filename=package://4_24_18_revel/meshes/link_5.STL; visual mesh filename=package://4_24_18_revel/meshes/link_5.STL
- link link_6: mass 0.222489248107418 -> 0.217466355310719; geometry collision mesh filename=package://4_24_18_revel/meshes/link_6.STL; visual mesh filename=package://4_24_18_revel/meshes/link_6.STL
Joints:
- joint finger_joint_1: axis -1 0 0 -> 0 -1 0
- joint finger_joint_2: axis -1 0 0 -> 0 -1 0
- joint joint_2: origin xyz=0.00038333 -0.0069353 0.10441 rpy=1.5708 0 0 -> xyz=0.00039444 -0.0064686 0.11076 rpy=1.5708 0 0
- joint joint_3: origin xyz=0 0.2224 0.014294 rpy=0 0 0 -> xyz=0 0.26625 0.014294 rpy=0 0 0
- joint joint_4: axis 0 -1 0 -> 0 0 1; limit lower=-2.5 upper=4.0 effort=10 velocity=1 -> lower=-4.5 upper=2.5 effort=10 velocity=1; origin xyz=0 0.19605 -0.015019 rpy=0 0 0 -> xyz=0 0.13713 -0.015019 rpy=-1.5708 0 0
- joint joint_5: origin xyz=0 0.08375 0.0040438 rpy=-1.5708 0 0 -> xyz=0 -0.0040438 0.086925 rpy=0 0 0
- joint joint_6: limit lower=0.5 upper=5.5 effort=10 velocity=1 -> lower=3.14 upper=7.85 effort=10 velocity=1; origin xyz=0 -0.019119 0.082 rpy=3.1416 0 1.5708 -> xyz=0 -0.019119 0.082 rpy=3.1416 0 3.1416

Commit message: updates to kinematics and joint limits

File: svenzva_description/robots/svenzva_arm.urdf (robot description, URDF)
Before this commit: robot revel, 11 links, 10 joints
Joints:
- joint joint_2: limit lower=-2.2 upper=2.2 effort=10 velocity=1 -> lower=-2.0 upper=2.0 effort=10 velocity=1
- joint joint_3: limit lower=-2.2 upper=2.2 effort=10 velocity=1 -> lower=-2.5 upper=2.5 effort=10 velocity=1
- joint joint_4: axis 0 0 1 -> 0 0 -1
- joint joint_5: limit lower=-1.7 upper=1.7 effort=10 velocity=1 -> lower=-1.8 upper=1.8 effort=10 velocity=1

Commit message: updates references to mesh

File: svenzva_description/robots/svenzva_arm.urdf (robot description, URDF)
Before this commit: robot revel, 11 links, 10 joints
Links:
- link base_link: geometry collision mesh filename=package://svenzva_description/meshes/base_link.STL; visual mesh filename=package://svenzva_description/meshes/base_link.STL
- link link_1: geometry collision mesh filename=package://svenzva_description/meshes/link_1.STL; visual mesh filename=package://svenzva_description/meshes/link_1.STL
- link link_2: geometry collision mesh filename=package://svenzva_description/meshes/link_2.STL; visual mesh filename=package://svenzva_description/meshes/link_2.STL
- link link_3: geometry collision mesh filename=package://svenzva_description/meshes/link_3.STL; visual mesh filename=package://svenzva_description/meshes/link_3.STL
- link link_4: geometry collision mesh filename=package://svenzva_description/meshes/link_4.STL; visual mesh filename=package://svenzva_description/meshes/link_4.STL
- link link_5: geometry collision mesh filename=package://svenzva_description/meshes/link_5.STL; visual mesh filename=package://svenzva_description/meshes/link_5.STL
- link link_6: geometry collision mesh filename=package://svenzva_description/meshes/link_6.STL; visual mesh filename=package://svenzva_description/meshes/link_6.STL
Joints:
- joint joint_6: limit lower=3.14 upper=7.85 effort=10 velocity=1 -> lower=0.0 upper=5.85 effort=10 velocity=1

Commit message: added dae textures

File: svenzva_description/robots/svenzva_arm.urdf (robot description, URDF)
Before this commit: robot revel, 11 links, 10 joints
Links:
- link base_link: geometry collision mesh filename=package://svenzva_description/meshes/base_link.STL; visual mesh filename=package://svenzva_description/textures/base_link.dae
- link link_1: geometry collision mesh filename=package://svenzva_description/meshes/link_1.STL; visual mesh filename=package://svenzva_description/textures/link_1.dae
- link link_2: geometry collision mesh filename=package://svenzva_description/meshes/link_2.STL; visual mesh filename=package://svenzva_description/textures/link_2.dae
- link link_3: geometry collision mesh filename=package://svenzva_description/meshes/link_3.STL; visual mesh filename=package://svenzva_description/textures/link_3.dae
- link link_4: geometry collision mesh filename=package://svenzva_description/meshes/link_4.STL; visual mesh filename=package://svenzva_description/textures/link_4.dae
- link link_5: geometry collision mesh filename=package://svenzva_description/meshes/link_5.STL; visual mesh filename=package://svenzva_description/textures/link_5.dae
- link link_6: geometry collision mesh filename=package://svenzva_description/meshes/link_6.STL; visual mesh filename=package://svenzva_description/textures/link_6.dae

Commit message: modified joint limit for shorter wrist cable

File: svenzva_description/robots/svenzva_arm.urdf (robot description, URDF)
Before this commit: robot revel, 11 links, 10 joints
Joints:
- joint joint_6: limit lower=0.0 upper=5.85 effort=10 velocity=1 -> lower=0.2 upper=3.14 effort=10 velocity=1

Commit message: adds greater flexibility for joint 6

File: svenzva_description/robots/svenzva_arm.urdf (robot description, URDF)
Before this commit: robot revel, 11 links, 10 joints
Joints:
- joint joint_6: limit lower=0.2 upper=3.14 effort=10 velocity=1 -> lower=0.2 upper=5.5 effort=10 velocity=1

Commit message: cleanup to make set default arm parameters. Adds in moveit config

File: svenzva_description/robots/svenzva_arm.urdf (robot description, URDF)
Before this commit: robot revel, 11 links, 10 joints
Links:
- removed link pen_holder_base_link
- removed link pen_holder_tip_link
- added link finger_link_1, mass 0.0220307791071739; collision mesh filename=package://svenzva_description/meshes/finger_standard.STL; visual mesh filename=package://svenzva_description/meshes/finger_standard.STL
- added link finger_link_2, mass 0.0220307791071739; collision mesh filename=package://svenzva_description/meshes/finger_standard.STL; visual mesh filename=package://svenzva_description/meshes/finger_standard.STL
Joints:
- removed joint pen_holder_joint
- removed joint pen_holder_tip_joint
- added joint finger_joint_1: type prismatic, parent link_6, child finger_link_1, origin xyz=0 0 -0.052002 rpy=-3.1416 0 3.1416, axis 0 -1 0, limit lower=0 upper=0.05 effort=100 velocity=10
- added joint finger_joint_2: type prismatic, parent link_6, child finger_link_2, origin xyz=0 0 -0.052002 rpy=-3.1416 0 3.1416, axis 0 1 0, limit lower=0 upper=0.05 effort=100 velocity=10

File: svenzva_description/robots/svenzva_arm.xacro (robot description, xacro)
@@ -6,5 +6,5 @@
    <!-- Set gripper's configurable options: finger type, gripper accessories, etc -->
    <xacro:property name="finger_type" value="${finger_tapped}" />
-   <xacro:property name="gripper_attachment" value="true"/>
+   <xacro:property name="gripper_attachment" value="false"/>
    <xacro:property name="svenzva_vacuum_gripper_attachment" value="false" />
    <xacro:property name="svenzva_pen_gripper_attachment" value="true" />

Commit message: adds new finger type, and ability to change fingers in xacro

File: svenzva_description/robots/svenzva_arm.urdf (robot description, URDF)
Before this commit: robot revel, 11 links, 10 joints
Links:
- link finger_link_1: geometry collision mesh filename=package://svenzva_description/meshes/accessories/finger_sta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; visual mesh filename=package://svenzva_description/meshes/accessories/finger_sta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
- link finger_link_2: geometry collision mesh filename=package://svenzva_description/meshes/accessories/finger_sta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; visual mesh filename=package://svenzva_description/meshes/accessories/finger_sta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

File: svenzva_description/robots/svenzva_arm.xacro (robot description, xacro)
@@ -4,6 +4,7 @@
    <xacro:property name="finger_standard" value="standard" />
    <xacro:property name="finger_tapped" value="standard_tapped" />
+   <xacro:property name="finger_center" value="center"/>
    <!-- Set gripper's configurable options: finger type, gripper accessories, etc -->
-   <xacro:property name="finger_type" value="${finger_tapped}" />
+   <xacro:property name="finger_type" value="${finger_standard}" />
    <xacro:property name="gripper_attachment" value="false"/>
    <xacro:property name="svenzva_vacuum_gripper_attachment" value="false" />
@@ -416,9 +417,9 @@
   </joint>
   <xacro:unless value="${gripper_attachment}">
-      <xacro:revel_finger parent="link_6" finger_number="1" mesh_path="package://svenzva_description/meshes/finger_standard.STL">
+      <xacro:revel_finger parent="link_6" finger_number="1" mesh_path="package://svenzva_description/meshes/accessories/finger_${finger_type}.STL">
           <origin xyz="0 0 -0.003175" rpy="0 0 ${H_PI}" />
           <axis xyz="0 -1 0" />
       </xacro:revel_finger>
-      <xacro:revel_finger parent="link_6" finger_number="2" mesh_path="package://svenzva_description/meshes/finger_standard.STL">
+      <xacro:revel_finger parent="link_6" finger_number="2" mesh_path="package://svenzva_description/meshes/accessories/finger_${finger_type}.STL">
           <origin xyz="0 0 -0.003175" rpy="0 0 -${H_PI}" />
           <axis xyz="0 1 0" />
