Commit message: additional changes to fingers to standarize their origin. adds additional finger type

File: svenzva_description/robots/accessories/fingers.xacro (robot description, xacro)
@@ -14,8 +14,6 @@
 				izz="9.60841591398502E-06" />
 		</inertial>
-		<visual>
-		  <origin
-			xyz="0 0 0"
-			rpy="0 0 -3.14159" />
+        <visual>
+		  <xacro:insert_block name="origin" />
 		  <geometry>
 			<mesh

File: svenzva_description/robots/svenzva_arm.urdf (robot description, URDF)
Before this commit: robot revel, 11 links, 10 joints
Links:
- removed link finger_joint_2
- added link finger_link_2, mass 0.0220307791071739; collision mesh filename=package://svenzva_description/meshes/finger_standard.STL; visual mesh filename=package://svenzva_description/meshes/finger_standard.STL
- link finger_link_1: geometry collision mesh filename=package://svenzva_description/meshes/finger_standard.STL; visual mesh filename=package://svenzva_description/meshes/finger_standard.STL
Joints:
- joint finger_joint_2: axis 0 -1 0 -> 0 1 0; child finger_joint_2 -> finger_link_2; limit lower=-0.05 upper=0 effort=100 velocity=10 -> lower=0 upper=0.05 effort=100 velocity=10

File: svenzva_description/robots/svenzva_arm.xacro (robot description, xacro)
@@ -5,4 +5,6 @@
    <xacro:property name="svenzva_vacuum_gripper_attachment" value="false" />
    <xacro:property name="svenzva_pen_gripper_attachment" value="false" />
+   <xacro:property name="H_PI" value="1.570796"/>
+   <xacro:property name="PI" value="3.14159"/>
    <!-- Set link name properties -->
    <xacro:property name="end_effector_link_name" value="ee_link"/>
@@ -422,9 +424,9 @@
   </joint>
   <xacro:revel_finger parent="link_6" finger_number="1" mesh_path="package://svenzva_description/meshes/finger_standard.STL">
-      <origin xyz="0 0 -0.00196" rpy="0 0 -3.14159" />
+      <origin xyz="0 0 -0.00492" rpy="0 0 ${H_PI}" />
       <axis xyz="0 -1 0" />
   </xacro:revel_finger>
   <xacro:revel_finger parent="link_6" finger_number="2" mesh_path="package://svenzva_description/meshes/finger_standard.STL">
-      <origin xyz="0 0 -0.00196" rpy="0 0 0" />
+      <origin xyz="0 0 -0.00492" rpy="0 0 -${H_PI}" />
       <axis xyz="0 1 0" />
   </xacro:revel_finger>

Commit message: additional offset changes to fingers for greater accuracy and modularity. adds two accessories

File: svenzva_description/robots/accessories/fingers.xacro (robot description, xacro)
@@ -38,6 +38,6 @@
 	  <joint name="finger_joint_${finger_number}" type="prismatic">
 		<origin
-		  xyz="0 0 -0.052509"
-		  rpy="-3.1416 -1.8964E-18 3.1416" />
+		  xyz="0 0 -0.052002"
+		  rpy="-3.1416 0 3.1416" />
 		<parent
             link="${parent}" />

File: svenzva_description/robots/accessories/pen_holder.xacro (robot description, xacro)
@@ -2,16 +2,36 @@
 <robot xmlns:xacro="http://ros.org/wiki/xacro" name="pen_holder">
     <xacro:macro name="pen_holder" params="parent *origin">
-		<joint name="pen_holder_joint" type="fixed">
-            <xacro:insert_block name="origin" />
-            <parent link="${parent}" />
-            <child link="pen_holder_link" />
-        </joint>
-	    <link name="pen_holder_link">
-			<visual>
-				<geometry>
-					<mesh filename="package://svenzva_description/meshes/accessories/pen_holder.STL" />
-				</geometry>
-			</visual>
-		</link>
+	<link name="pen_holder_base_link">
+    <visual>
+	  <xacro:insert_block name="origin"/>
+      <geometry>
+          <mesh filename="package://svenzva_description/textures/accessories/finger_pen_holder.dae"/>
+      </geometry>
+      <material
+        name="">
+        <color
+          rgba="0.898039215686275 0.917647058823529 0.929411764705882 1" />
+      </material>
+    </visual>
+    <collision>
+		<xacro:insert_block name="origin"/>
+      <geometry>
+        <mesh filename="package://svenzva_description/meshes/accessories/finger_pen_holder.STL"/>
+      </geometry>
+    </collision>
+    </link>
+    <joint name="pen_holder_joint" type="fixed">
+		<origin xyz="0 0 -0.052002" rpy="-3.1416 0 3.1416" />
+		<parent link="${parent}" />
+		<child link="pen_holder_base_link" />
+	</joint>
+	<link name="pen_holder_tip_link">
+		<origin xyz="0 0 0.16" rpy="0 0 0"/>
+	</link>
+	<joint name="pen_holder_tip_joint" type="fixed">
+		<origin xyz="0 0 0.16" rpy="0 0 0" />
+		<parent link="pen_holder_base_link" />
+		<child link="pen_holder_tip_link" />
+	</joint>
     </xacro:macro>
 </robot>

File: svenzva_description/robots/accessories/vacuum_holder.xacro (robot description, xacro)
@@ -2,16 +2,44 @@
 <robot xmlns:xacro="http://ros.org/wiki/xacro" name="vacuum_holder">
     <xacro:macro name="vacuum_holder" params="parent *origin">
-		<joint name="vacuum_holder_joint" type="fixed">
-            <xacro:insert_block name="origin" />
-            <parent link="${parent}" />
-            <child link="vacuum_holder_link" />
-        </joint>
-	    <link name="vacuum_holder_link">
-			<visual>
-				<geometry>
-					<mesh filename="package://svenzva_description/meshes/accessories/vacuum_holder.STL" />
-				</geometry>
-			</visual>
-		</link>
+	<link name="vacuum_holder_base_link">
+    <visual>
+	  <xacro:insert_block name="origin"/>
+      <geometry>
+          <mesh filename="package://svenzva_description/textures/accessories/vacuum_holder.dae"/>
+      </geometry>
+      <material
+        name="">
+        <color
+          rgba="0.898039215686275 0.917647058823529 0.929411764705882 1" />
+      </material>
+    </visual>
+    <collision>
+		<xacro:insert_block name="origin"/>
+      <geometry>
+        <mesh filename="package://svenzva_description/meshes/accessories/vacuum_holder.STL"/>
+      </geometry>
+    </collision>
+    </link>
+    <joint name="vacuum_holder_joint" type="fixed">
+		<origin xyz="0 0 -0.052002" rpy="-3.1416 0 3.1416" />
+		<parent link="${parent}" />
+		<child link="vacuum_holder_base_link" />
+	</joint>
+	<link name="vacuum_holder_suction_base_link">
+		<origin xyz="0 0 0.16" rpy="0 0 0"/>
+	</link>
+	<joint name="vacuum_holder_suction_base_joint" type="fixed">
+		<origin xyz="0 0 0.0591" rpy="0 0 0" />
+		<parent link="vacuum_holder_base_link" />
+		<child link="vacuum_holder_suction_base_link" />
+	</joint>
+	<link name="vacuum_holder_suction_tip_link">
+		<origin xyz="0 0 0.16" rpy="0 0 0"/>
+	</link>
+	<joint name="vacuum_holder_suction_tip_joint" type="fixed">
+		<origin xyz="0 0 0.0125" rpy="0 0 0" />
+		<parent link="vacuum_holder_suction_base_link" />
+		<child link="vacuum_holder_suction_tip_link" />
+	</joint>
     </xacro:macro>
 </robot>

File: svenzva_description/robots/svenzva_arm.urdf (robot description, URDF)
Before this commit: robot revel, 11 links, 10 joints
Links:
- removed link finger_link_1
- removed link finger_link_2
- added link pen_holder_base_link; collision mesh filename=package://svenzva_description/meshes/accessories/finger_pen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; visual mesh filename=package://svenzva_description/meshes/accessories/finger_pen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
- added link pen_holder_tip_link
Joints:
- removed joint finger_joint_1
- removed joint finger_joint_2
- added joint pen_holder_joint: type fixed, parent link_6, child pen_holder_base_link, origin xyz=0 0 -0.052002 rpy=-3.1416 0 3.1416
- added joint pen_holder_tip_joint: type fixed, parent pen_holder_base_link, child pen_holder_tip_link, origin xyz=0 0 0.16 rpy=0 0 0

File: svenzva_description/robots/svenzva_arm.xacro (robot description, xacro)
@@ -1,12 +1,15 @@
 <?xml version="1.0"?>
 <robot name="revel" xmlns:xacro="http://ros.org/wiki/xacro">
+   <!-- Finger constants -->
+   <xacro:property name="finger_standard" value="standard" />
+   <xacro:property name="finger_tapped" value="standard_tapped" />
    <!-- Set gripper's configurable options: finger type, gripper accessories, etc -->
-   <xacro:property name="finger_type" value="standard" />
+   <xacro:property name="finger_type" value="${finger_tapped}" />
+   <xacro:property name="gripper_attachment" value="true"/>
    <xacro:property name="svenzva_vacuum_gripper_attachment" value="false" />
-   <xacro:property name="svenzva_pen_gripper_attachment" value="false" />
+   <xacro:property name="svenzva_pen_gripper_attachment" value="true" />
    <xacro:property name="H_PI" value="1.570796"/>
    <xacro:property name="PI" value="3.14159"/>
    <!-- Set link name properties -->
-   <xacro:property name="end_effector_link_name" value="ee_link"/>
    <!-- Set filepath constants -->
    <xacro:property name="finger_mesh_path" value="package://svenzva_description/meshes/finger_joint_2.STL" />
@@ -14,15 +17,4 @@
    <xacro:include filename="$(find svenzva_description)/robots/accessories/pen_holder.xacro" />
    <xacro:include filename="$(find svenzva_description)/robots/accessories/fingers.xacro" />
-   <!-- Reason about accessory inclusion -->
-   <xacro:if value="${svenzva_vacuum_gripper_attachment}">
-        <xacro:vacuum_holder parent="ee_link">
-            <origin xyz="0 0 0" rpy="0 0 0" />
-        </xacro:vacuum_holder>
-   </xacro:if>
-   <xacro:if value="${svenzva_pen_gripper_attachment}">
-       <xacro:pen_holder parent="ee_link">
-            <origin xyz="0 0 0" rpy="0 0 0" />
-        </xacro:pen_holder>
-   </xacro:if>
    <gazebo>
      <plugin name="gazebo_ros_control" filename="libgazebo_ros_control.so">
@@ -423,16 +415,30 @@
       velocity="1" />
   </joint>
-  <xacro:revel_finger parent="link_6" finger_number="1" mesh_path="package://svenzva_description/meshes/finger_standard.STL">
-      <origin xyz="0 0 -0.00492" rpy="0 0 ${H_PI}" />
-      <axis xyz="0 -1 0" />
-  </xacro:revel_finger>
-  <xacro:revel_finger parent="link_6" finger_number="2" mesh_path="package://svenzva_description/meshes/finger_standard.STL">
-      <origin xyz="0 0 -0.00492" rpy="0 0 -${H_PI}" />
-      <axis xyz="0 1 0" />
-  </xacro:revel_finger>
-  <link name="${end_effector_link_name}"> </link>
+  <xacro:unless value="${gripper_attachment}">
+      <xacro:revel_finger parent="link_6" finger_number="1" mesh_path="package://svenzva_description/meshes/finger_standard.STL">
+          <origin xyz="0 0 -0.003175" rpy="0 0 ${H_PI}" />
+          <axis xyz="0 -1 0" />
+      </xacro:revel_finger>
+      <xacro:revel_finger parent="link_6" finger_number="2" mesh_path="package://svenzva_description/meshes/finger_standard.STL">
+          <origin xyz="0 0 -0.003175" rpy="0 0 -${H_PI}" />
+          <axis xyz="0 1 0" />
+      </xacro:revel_finger>
+  </xacro:unless>
+  <xacro:if value="${gripper_attachment}">
+      <xacro:if value="${svenzva_pen_gripper_attachment}">
+        <xacro:pen_holder parent="link_6">
+            <origin xyz="0 0 -0.003175" rpy="0 0 -${H_PI}" />
+        </xacro:pen_holder>
+      </xacro:if>
+      <xacro:if value="${svenzva_vacuum_gripper_attachment}">
+          <xacro:vacuum_holder parent="link_6">
+            <origin xyz="0 0 -0.003175" rpy="0 0 -${H_PI}" />
+        </xacro:vacuum_holder>
+      </xacro:if>
+  </xacro:if>
+  <link name="ee_link"> </link>
   <joint name="ee_joint" type="fixed">
     <parent link="link_6"/>
-    <child link="${end_effector_link_name}"/>
+    <child link="ee_link"/>
     <origin xyz="0 0 -0.05" rpy="3.14159 0 0"/>
   </joint>
